File: PCBs/solenoid_controller/solenoid controller.kicad_pcb (KiCad board)
At the start: 2 copper layers, 100 x 65 mm, 63 parts, among them J1 Conn_02x03_Odd_Even, J2 Conn_02x03_Odd_Even, J3 Conn_02x04_Odd_Even, J4 SWD, J5 Solenoid, Q1 Q_NMOS_SDG, U1 23LCV512, U2 AMS1117-3.3, U3 AOZ1284, U4 AMS1117-5.0, U5 STM32F030K6Tx, U6 MIC4416, U7 ACS712xLCTR-30A, Y1 12Mhz

Commit message: PCB update
Parts:
- added J6: GND_CONN, My_elements:single_PAD, F.Cu at (161.2, 131.4)
- added J7: 28V_CONN, My_elements:single_PAD, F.Cu at (163.3, 73.8)
- added R17: 1k, Resistor_SMD:R_0603_1608Metric_Pad0.98x0.95mm_HandSolder, F.Cu at (138.3, 85.5)
- C1, C2, C3, C4, C5: moved to B.Cu
- C13, C15, C18, C8: footprint Capacitor_SMD:C_0603_1608Metric_Pad1.08x0.95mm_HandSolder -> Capacitor_SMD:C_0805_2012Metric_Pad1.18x1.45mm_HandSolder
- D7: footprint Diode_SMD:D_SMA -> Diode_SMD:D_SMA_Handsoldering
- R1: value 22k -> 10k
- moved C14 185.4 mm to (98.8, 119.6), turned to 180 degrees
- moved R2 178.6 mm to (105.8, 132.5)
- moved R1 176.8 mm to (110.0, 132.5)
- moved R6 165.5 mm to (97.7, 130.3)
- moved C12 165.5 mm to (103.1, 119.6), turned to 180 degrees
- moved C3 160.1 mm to (111.5, 120.1), turned to 180 degrees
- moved JP1 159.5 mm to (98.2, 81.2), turned to -90 degrees
- moved C11 157.1 mm to (104.5, 112.6)
- moved D3 156.4 mm to (94.1, 130.3)
- moved D1 153.8 mm to (107.1, 98.9), turned to 180 degrees
- moved C20 151.5 mm to (133.6, 121.3), turned to -90 degrees
- moved C4 151.4 mm to (111.5, 118.4), turned to 180 degrees
- moved C7 150.8 mm to (111.7, 79.6), turned to 180 degrees
- moved C5 148.0 mm to (111.5, 121.8), turned to 180 degrees
- moved D4 147.5 mm to (94.1, 132.0)
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Connections:
- C11 pad 1: Net-(C11-Pad1) -> Net-(U5-PF0)
- C14 pad 1: Net-(C11-Pad1) -> Net-(U5-PF1)
- JP2 pad 2: +5VP -> Net-(JP2-B)
- U5 pad 2: Net-(U5-Pad2) -> Net-(U5-PF0)
- U5 pad 3: Net-(C11-Pad1) -> Net-(U5-PF1)
- Y1 pad 1: Net-(C11-Pad1) -> Net-(U5-PF1)
- Y1 pad 3: Net-(U5-Pad2) -> Net-(U5-PF0)
Routing:
- net /HALL_OUT: track 0.00 -> 73.8 mm, vias 0 -> 2
- net /S_TX: track 0.00 -> 70.3 mm, vias 0 -> 4
- net /S_RX: track 0.00 -> 68.3 mm, vias 0 -> 3
- net /MOSFET_VOL_DIV: track 0.00 -> 68.0 mm, vias 0 -> 5
- net +12V: track 0.00 -> 53.5 mm, vias 0 -> 5
- net /PROX_22: track 0.00 -> 48.4 mm, vias 0 -> 3
- net /PROX_21: track 0.00 -> 47.4 mm, vias 0 -> 3
- net /PROX_23: track 0.00 -> 46.4 mm, vias 0 -> 2
- net +28V: track 0.00 -> 43.8 mm
- net +3V3: track 0.00 -> 36.7 mm, vias 0 -> 3
- net Net-(J5-Pin_1): track 0.00 -> 32.5 mm
- net Net-(D7-A): track 0.00 -> 31.6 mm
- net Net-(D5-K): track 0.00 -> 29.3 mm
- net /PROX_13: track 0.00 -> 25.6 mm, vias 0 -> 1
- net /PROX_12: track 0.00 -> 23.8 mm, vias 0 -> 1
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- added copper zone on F.Cu, net GND
Other:
- board size 100 x 65 mm -> 87.9 x 65 mm

Commit message: solenoid controller finished
Parts:
- removed Q1: Q_NMOS_SDG, Package_TO_SOT_SMD:TO-263-2
- added Q2: Q_NMOS_GDS, Package_TO_SOT_SMD:TO-263-2, F.Cu at (154.2, 119.0)
- added REF**: MountingHole_2.2mm_M2, MountingHole:MountingHole_2.2mm_M2, F.Cu at (137.5, 75.0)
- added REF**: MountingHole_2.2mm_M2, MountingHole:MountingHole_2.2mm_M2, F.Cu at (137.5, 132.5)
- added REF**: MountingHole_2.2mm_M2, MountingHole:MountingHole_2.2mm_M2, F.Cu at (120.0, 75.0)
- added SW1: SW_Push, Button_Switch_SMD:SW_SPST_TL3342, F.Cu at (100.6, 75.2)
- moved D4 24.4 mm to (118.5, 132.7), turned to 90 degrees
- moved D3 22.9 mm to (116.8, 132.7), turned to 90 degrees
- moved R7 21.0 mm to (118.5, 129.2), turned to 90 degrees
- moved R6 19.2 mm to (116.8, 129.2), turned to 90 degrees
- moved JP1 3.97 mm to (102.1, 80.6)
- moved R14 3.79 mm to (136.3, 121.5)
- moved C7 1.40 mm to (111.7, 81.0)
- moved C19 0.13 mm to (134.3, 89.0)
- moved C1 0.10 mm to (114.0, 119.3)
Routing:
- net +12V: track 53.5 -> 186.9 mm, vias 5 -> 13
- net +3V3: track 36.7 -> 158.6 mm, vias 3 -> 7
- net /NRST: track 6.55 -> 83.0 mm, vias 2 -> 7
- net /SWDIO: track 0.00 -> 70.4 mm, vias 0 -> 4
- net /BUCK_VOL_DIV: track 9.38 -> 79.4 mm, vias 0 -> 7
- net +5VP: track 0.00 -> 68.5 mm, vias 0 -> 2
- net /SWCLK: track 0.00 -> 66.5 mm, vias 0 -> 4
- net /MOSFET_VOL_DIV: track 68.0 -> 124.8 mm, vias 5 -> 7
- net +5V: track 21.9 -> 75.3 mm, vias 2 -> 6
- net GND: track 11.6 -> 60.9 mm, vias 4 -> 38
- net /BUCK_ENABLE: track 11.6 -> 55.5 mm, vias 0 -> 2
- net Net-(J5-Pin_1): track 32.5 -> 57.3 mm, vias 0 -> 2
- net Net-(J3-Pin_1): track 0.00 -> 19.0 mm, vias 0 -> 1
- net /MOSFET_CTRL: track 0.00 -> 17.3 mm, vias 0 -> 2
- net Net-(U5-PB6): track 0.00 -> 16.8 mm, vias 0 -> 2
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- added copper zone on B.Cu, net GND
Other:
- board size 87.9 x 65 mm -> 88.1 x 64.9 mm
